File: Eagle/obsolete/MS20v2.sch (EAGLE design)
At the start: 62 parts, among them IC1 LM13700M, IC2 TL074D, T1 2N3906, T2 2N3906

Commit message: updated drawing for readability
Connections:
- net N$1: now also D2.C; no longer D2.A
- net N$2: now also D1.A; no longer D1.C
- net N$5: now also D1.C; no longer D1.A
- net N$8: now also D2.A; no longer D2.C
Other:
- moved on the sheet: ATRIM, C1, C10, C2, C4, C6, C7, C8, C9, CON1, CV1, CV2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
